Commit message: Fix collision of sample.urdf

File: sample.urdf (robot description, URDF)
Before this commit: robot robo, 13 links, 12 joints
Links:
- link l_elbow1: geometry collision box size=0.1 0.1 0.2; visual box size=0.1 0.1 0.2
- link l_shoulder1: geometry collision box size=0.1 0.1 0.1; visual box size=0.1 0.1 0.1
- link l_shoulder2: geometry collision box size=0.1 0.1 0.1; visual box size=0.1 0.1 0.1
- link l_shoulder3: geometry collision box size=0.1 0.1 0.2; visual box size=0.1 0.1 0.2
- link l_wrist1: geometry collision box size=0.1 0.15 0.1; visual box size=0.1 0.15 0.1
- link l_wrist2: geometry collision box size=0.05 0.08 0.15; visual box size=0.05 0.08 0.15
- link r_elbow1: geometry collision box size=0.1 0.1 0.2; visual box size=0.1 0.1 0.2
- link r_shoulder1: geometry collision box size=0.1 0.1 0.1; visual box size=0.1 0.1 0.1
- link r_shoulder2: geometry collision box size=0.1 0.1 0.1; visual box size=0.1 0.1 0.1
- link r_shoulder3: geometry collision box size=0.1 0.1 0.2; visual box size=0.1 0.1 0.2
- link r_wrist1: geometry collision box size=0.1 0.15 0.1; visual box size=0.1 0.15 0.1
- link r_wrist2: geometry collision box size=0.05 0.08 0.15; visual box size=0.05 0.08 0.15
- link root: geometry collision box size=0.2 0.2 0.4; visual box size=0.2 0.2 0.4

Commit message: Change the sample.urdf to single arm robot

File: sample.urdf (robot description, URDF)
Before this commit: robot robo, 13 links, 12 joints
Links:
- removed link r_elbow1
- removed link r_shoulder1
- removed link r_shoulder2
- removed link r_shoulder3
- removed link r_wrist1
- removed link r_wrist2
Joints:
- removed joint r_elbow_pitch
- removed joint r_shoulder_pitch
- removed joint r_shoulder_roll
- removed joint r_shoulder_yaw
- removed joint r_wrist_pitch
- removed joint r_wrist_yaw
- joint l_elbow_pitch: limit lower=-2 upper=1.0 effort=0 velocity=1.0 -> lower=-2.0 upper=0.5 effort=0 velocity=1.0
- joint l_shoulder_pitch: limit lower=-1 upper=1.0 effort=0 velocity=1.0 -> lower=-2.0 upper=0.5 effort=0 velocity=1.0
- joint l_shoulder_roll: limit lower=-2 upper=1.0 effort=0 velocity=1.0 -> lower=-1 upper=2.0 effort=0 velocity=1.0
- joint l_wrist_pitch: limit lower=-2 upper=1.0 effort=0 velocity=1.0 -> lower=-2 upper=2.0 effort=0 velocity=1.0
- joint l_wrist_yaw: limit lower=-2 upper=1.0 effort=0 velocity=1.0 -> lower=-1 upper=1.0 effort=0 velocity=1.0

Commit message: improve ik, play, add smooth

File: sample.urdf (robot description, URDF)
Before this commit: robot robo, 7 links, 6 joints
Joints:
- joint l_elbow_pitch: limit lower=-2.0 upper=0.5 effort=0 velocity=1.0 -> lower=-2.0 upper=1.5 effort=0 velocity=1.0
- joint l_shoulder_pitch: limit lower=-2.0 upper=0.5 effort=0 velocity=1.0 -> lower=-2.0 upper=1.5 effort=0 velocity=1.0
- joint l_shoulder_roll: limit lower=-1 upper=2.0 effort=0 velocity=1.0 -> lower=-1.5 upper=2.0 effort=0 velocity=1.0
- joint l_shoulder_yaw: limit lower=-1 upper=1.0 effort=0 velocity=1.0 -> lower=-1.5 upper=1.5 effort=0 velocity=1.0
- joint l_wrist_yaw: limit lower=-1 upper=1.0 effort=0 velocity=1.0 -> lower=-1.5 upper=1.5 effort=0 velocity=1.0

Commit message: Adjust sample.urdf and reach.rs
* make longer arm in sample.urdf
* re-arrange obstacles and the target

File: sample.urdf (robot description, URDF)
Before this commit: robot robo, 7 links, 6 joints
Links:
- link l_elbow1: geometry collision box size=0.25 0.05 0.1; visual box size=0.25 0.05 0.1
- link l_shoulder3: geometry collision box size=0.25 0.1 0.15; visual box size=0.25 0.1 0.15
- link l_wrist1: geometry collision box size=0.25 0.15 0.1; visual box size=0.25 0.15 0.1
- link l_wrist2: geometry collision box size=0.20 0.08 0.05; visual box size=0.20 0.08 0.05
- link root: geometry collision box size=0.2 0.2 0.6; visual box size=0.2 0.2 0.6
Joints:
- joint l_elbow_pitch: origin xyz=0.0 0.0 -0.2 -> xyz=0.3 0.0 0.0
- joint l_shoulder_yaw: origin xyz=0.0 0.2 0.2 -> xyz=0.0 0.2 0.5
- joint l_wrist_pitch: origin xyz=0.0 0.0 -0.2 -> xyz=0.1 0.0 0.0
- joint l_wrist_yaw: origin xyz=0.0 0.0 -0.2 -> xyz=0.3 0.0 0.0

Commit message: Set end link name explicitly in reach.rs to support grippers

File: sample.urdf (robot description, URDF)
Before this commit: robot robo, 7 links, 6 joints
Links:
- added link l_gripper1; collision cylinder length=0.15 radius=0.02; visual cylinder length=0.15 radius=0.02
- added link l_gripper2; collision cylinder length=0.15 radius=0.02; visual cylinder length=0.15 radius=0.02
- link l_wrist2: geometry collision box size=0.1 0.08 0.05; visual box size=0.1 0.08 0.05
Joints:
- added joint l_gripper_linear1: type prismatic, parent l_wrist2, child l_gripper1, origin xyz=0.15 -0.05 0.0 rpy=0 0 1.57, axis 1 0 0, limit lower=-0.05 upper=0.05 effort=0 velocity=1.0
- added joint l_gripper_linear2: type prismatic, parent l_wrist2, child l_gripper2, origin xyz=0.15 0.05 0.0 rpy=0 0 1.57, axis 1 0 0, limit lower=-0.05 upper=0.05 effort=0 velocity=1.0
- joint l_wrist_pitch: origin xyz=0.1 0.0 0.0 -> xyz=0.15 0.0 0.0
- joint l_wrist_yaw: origin xyz=0.3 0.0 0.0 -> xyz=0.25 0.0 0.0

Commit message: Update sample.urdf
* add l_tool link
* fix gripper rotation

File: sample.urdf (robot description, URDF)
Before this commit: robot robo, 9 links, 8 joints
Links:
- added link l_tool; visual box size=0.01 0.01 0.01
Joints:
- added joint l_tool_fixed: type fixed, parent l_wrist2, child l_tool, origin xyz=0.2 0.0 0.0

Commit message: Update dependency to support mimic joint

File: sample.urdf (robot description, URDF)
Before this commit: robot robo, 10 links, 9 joints
Joints:
- joint l_gripper_linear2: mimic (none) -> joint=l_gripper_linear1 multiplier=-1.0
